File: src/RepRap Display Controller.kicad_pcb (KiCad board)
At the start: 2 copper layers, 17.8 x 43.2 mm, 8 parts, among them J1 EXP1, J2 EXP2, P1 Digital, P2 Analog, P3 CONN_01X01, P4 CONN_01X01, P5 CONN_01X01, P6 CONN_01X01

Commit message: Reorganization and Klipper Config
Files organized into folders for ease of navigation. Also added an UNTESTED Klipper .cfg file that can be included into the main printer.cfg to enable this disaply adaptor.
Other:
- board text added: "ICSP"
- board text added: "USB"
Changed lines of the file:
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@@
   (general
     (thickness 1.6)
-    (drawings 29)
+    (drawings 44)
     (tracks 73)
     (zones 0)
@@
     (38 B.Mask user)
     (39 F.Mask user)
-    (40 Dwgs.User user hide)
+    (40 Dwgs.User user)
     (41 Cmts.User user)
     (42 Eco1.User user)
@@
     (44 Edge.Cuts user)
     (45 Margin user)
-    (46 B.CrtYd user hide)
-    (47 F.CrtYd user hide)
-    (48 B.Fab user hide)
-    (49 F.Fab user hide)
+    (46 B.CrtYd user)
+    (47 F.CrtYd user)
+    (48 B.Fab user)
+    (49 F.Fab user)
   )
   (setup
@@
     (visible_elements 7FFFFFFF)
     (pcbplotparams
-      (layerselection 0x00030_80000001)
+      (layerselection 0x010f0_ffffffff)
       (usegerberextensions false)
       (usegerberattributes false)
@@
       (outputformat 1)
       (mirror false)
-      (drillshape 1)
+      (drillshape 0)
       (scaleselection 1)
-      (outputdirectory ""))
+      (outputdirectory "../Gerbers/"))
   )
   (net 0 "")
@@
     (pad 1 thru_hole circle (at 0 0) (size 2.54 2.54) (drill 1.778) (layers *.Cu *.Mask F.SilkS))
   )
+  (gr_line (start 150.622 106.172) (end 150.622 110.363) (layer F.SilkS) (width 0.15))
+  (gr_line (start 143.51 106.172) (end 150.622 106.172) (layer F.SilkS) (width 0.15))
+  (gr_line (start 143.51 110.363) (end 143.51 106.172) (layer F.SilkS) (width 0.15))
+  (gr_line (start 150.622 110.363) (end 143.51 110.363) (layer F.SilkS) (width 0.15))
+  (gr_line (start 150.876 67.7545) (end 143.256 67.7545) (layer F.SilkS) (width 0.15))
+  (gr_line (start 150.876 72.517) (end 150.876 67.7545) (layer F.SilkS) (width 0.15))
+  (gr_line (start 143.256 72.517) (end 150.876 72.517) (layer F.SilkS) (width 0.15))
+  (gr_line (start 143.256 67.7545) (end 143.256 72.517) (layer F.SilkS) (width 0.15))
+  (gr_circle (center 147.574 86.487) (end 147.574 85.725) (layer F.SilkS) (width 0.15))
+  (gr_line (start 149.479 85.217) (end 145.542 85.217) (layer F.SilkS) (width 0.15))
+  (gr_line (start 149.479 87.757) (end 149.479 85.217) (layer F.SilkS) (width 0.15))
+  (gr_line (start 145.542 87.757) (end 149.479 87.757) (layer F.SilkS) (width 0.15))
+  (gr_line (start 145.542 85.217) (end 145.542 87.757) (layer F.SilkS) (width 0.15))
+  (gr_text ICSP (at 147.066 70.231) (layer F.SilkS)
+    (effects (font (size 1.5 1.5) (thickness 0.15)))
+  )
+  (gr_text USB (at 147.066 108.331) (layer F.SilkS)
+    (effects (font (size 2 2) (thickness 0.3)))
+  )
   (gr_text EXP1 (at 152.654 78.232 90) (layer B.SilkS)
