File: KiCad/RepRap Display Controller.kicad_pcb (KiCad board)
At the start: 2 copper layers, 17.8 x 43.2 mm, 8 parts, among them J1 EXP1, J2 EXP2, P1 Digital, P2 Analog, P3 CONN_01X01, P4 CONN_01X01, P5 CONN_01X01, P6 CONN_01X01

Commit message: Added license and versioning to PCB
Added V1.0 to board for proper versioning going forward and CC BY-NC license.

Basically, Full reign to share and modify as long as it is NOT used commercial and retains all attribution to the source.
Parts:
- added G***: LOGO, TRA_KiCad_Footprints:VoronDesign_Text_35x20, F.Cu at (142.6, 89.0)
- added G***: LOGO, TRA_KiCad_Footprints:VoronLogo_6pt5mm_silkScreen, F.Cu at (149.0, 89.0)
Other:
- board text added: "ICSP"
- board text added: "Tim Abraham"
- board text added: "USB"
- board text added: "V1.0"
